Commit message: Updated ee_desciption to tools_description

File: intera_tools_description/urdf/electric_gripper/example_end_effector.urdf.xacro (robot description, xacro)
@@ -1,5 +1,5 @@
 <?xml version="1.0"?>
 <robot xmlns:xacro="http://www.ros.org/wiki/xacro" name="left_electric_gripper">
-  <xacro:include filename="$(find rethink_ee_description)/urdf/electric_gripper/rethink_electric_gripper.xacro" />
+  <xacro:include filename="$(find intera_tools_description)/urdf/electric_gripper/rethink_electric_gripper.xacro" />
   <xacro:rethink_electric_gripper side="left"
                                   l_finger="extended_narrow"

File: intera_tools_description/urdf/electric_gripper/fingers/basic_hard_tip.xacro (robot description, xacro)
@@ -10,5 +10,5 @@
         <origin rpy="0 0 ${pi*(g_reflect+1)/2}" xyz="0 0 0"/>
         <geometry>
-          <mesh filename="package://rethink_ee_description/meshes/electric_gripper/fingers/basic_hard_tip.DAE" />
+          <mesh filename="package://intera_tools_description/meshes/electric_gripper/fingers/basic_hard_tip.DAE" />
         </geometry>
       </visual>

File: intera_tools_description/urdf/electric_gripper/fingers/basic_soft_tip.xacro (robot description, xacro)
@@ -10,5 +10,5 @@
         <origin rpy="0 0 ${pi*(g_reflect+1)/2}" xyz="0 0 0"/>
         <geometry>
-          <mesh filename="package://rethink_ee_description/meshes/electric_gripper/fingers/basic_soft_tip.DAE" />
+          <mesh filename="package://intera_tools_description/meshes/electric_gripper/fingers/basic_soft_tip.DAE" />
         </geometry>
       </visual>

File: intera_tools_description/urdf/electric_gripper/fingers/extended_narrow.xacro (robot description, xacro)
@@ -8,5 +8,5 @@
         <origin rpy="0 0 ${-pi/2*(reflect+1)}" xyz="0 0 0"/>
         <geometry>
-          <mesh filename="package://rethink_ee_description/meshes/electric_gripper/fingers/extended_narrow.DAE" />
+          <mesh filename="package://intera_tools_description/meshes/electric_gripper/fingers/extended_narrow.DAE" />
         </geometry>
       </visual>
@@ -46,5 +46,5 @@
      <xacro:property name="finger_tip" value="none" scope="local"/>
    </xacro:if>
-   <xacro:include filename="$(find rethink_ee_description)/urdf/electric_gripper/fingers/${finger_tip}.xacro" />
+   <xacro:include filename="$(find intera_tools_description)/urdf/electric_gripper/fingers/${finger_tip}.xacro" />
    <xacro:finger_tip_xacro parent_link="${gripper_side}_gripper_${finger_side}_finger" reflect="${reflect}" grasp="${finger_grasp}">
        <origin rpy="0 0 0" xyz="0.0 ${reflect*finger_width} ${finger_length}"/>

File: intera_tools_description/urdf/electric_gripper/fingers/extended_wide.xacro (robot description, xacro)
@@ -8,5 +8,5 @@
         <origin rpy="0 0 ${-pi/2*(reflect+1)}" xyz="0 0 0"/>
         <geometry>
-          <mesh filename="package://rethink_ee_description/meshes/electric_gripper/fingers/extended_wide.DAE" />
+          <mesh filename="package://intera_tools_description/meshes/electric_gripper/fingers/extended_wide.DAE" />
         </geometry>
       </visual>
@@ -46,5 +46,5 @@
      <xacro:property name="finger_tip" value="none" scope="local"/>
    </xacro:if>
-   <xacro:include filename="$(find rethink_ee_description)/urdf/electric_gripper/fingers/${finger_tip}.xacro" />
+   <xacro:include filename="$(find intera_tools_description)/urdf/electric_gripper/fingers/${finger_tip}.xacro" />
    <xacro:finger_tip_xacro parent_link="${gripper_side}_gripper_${finger_side}_finger" reflect="${reflect}" grasp="${finger_grasp}">
        <origin rpy="0 0 0" xyz="0.0 ${reflect*finger_width} ${finger_length}"/>

File: intera_tools_description/urdf/electric_gripper/fingers/half_round_tip.xacro (robot description, xacro)
@@ -10,5 +10,5 @@
         <origin rpy="0 0 ${pi*(g_reflect+1)/2}" xyz="0 0 0"/>
         <geometry>
-          <mesh filename="package://rethink_ee_description/meshes/electric_gripper/fingers/half_round_tip.DAE" />
+          <mesh filename="package://intera_tools_description/meshes/electric_gripper/fingers/half_round_tip.DAE" />
         </geometry>
       </visual>

File: intera_tools_description/urdf/electric_gripper/fingers/paddle_tip.xacro (robot description, xacro)
@@ -10,5 +10,5 @@
         <origin rpy="0 0 ${pi*(g_reflect+1)/2}" xyz="0 0 0"/>
         <geometry>
-          <mesh filename="package://rethink_ee_description/meshes/electric_gripper/fingers/paddle_tip.DAE" />
+          <mesh filename="package://intera_tools_description/meshes/electric_gripper/fingers/paddle_tip.DAE" />
         </geometry>
       </visual>

File: intera_tools_description/urdf/electric_gripper/fingers/standard_narrow.xacro (robot description, xacro)
@@ -8,5 +8,5 @@
         <origin rpy="0 0 ${-pi/2*(reflect+1)}" xyz="0 0 0"/>
         <geometry>
-          <mesh filename="package://rethink_ee_description/meshes/electric_gripper/fingers/standard_narrow.DAE" />
+          <mesh filename="package://intera_tools_description/meshes/electric_gripper/fingers/standard_narrow.DAE" />
         </geometry>
       </visual>
@@ -46,5 +46,5 @@
      <xacro:property name="finger_tip" value="none" scope="local"/>
    </xacro:if>
-   <xacro:include filename="$(find rethink_ee_description)/urdf/electric_gripper/fingers/${finger_tip}.xacro" />
+   <xacro:include filename="$(find intera_tools_description)/urdf/electric_gripper/fingers/${finger_tip}.xacro" />
    <xacro:finger_tip_xacro parent_link="${gripper_side}_gripper_${finger_side}_finger" reflect="${reflect}" grasp="${finger_grasp}">
        <origin rpy="0 0 0" xyz="0.0 ${reflect*finger_width} ${finger_length}"/>

File: intera_tools_description/urdf/electric_gripper/fingers/standard_wide.xacro (robot description, xacro)
@@ -8,5 +8,5 @@
         <origin rpy="0 0 ${-pi/2*(reflect+1)}" xyz="0 0 0"/>
         <geometry>
-          <mesh filename="package://rethink_ee_description/meshes/electric_gripper/fingers/standard_wide.DAE" />
+          <mesh filename="package://intera_tools_description/meshes/electric_gripper/fingers/standard_wide.DAE" />
         </geometry>
       </visual>
@@ -46,5 +46,5 @@
      <xacro:property name="finger_tip" value="none" scope="local"/>
    </xacro:if>
-   <xacro:include filename="$(find rethink_ee_description)/urdf/electric_gripper/fingers/${finger_tip}.xacro" />
+   <xacro:include filename="$(find intera_tools_description)/urdf/electric_gripper/fingers/${finger_tip}.xacro" />
    <xacro:finger_tip_xacro parent_link="${gripper_side}_gripper_${finger_side}_finger" reflect="${reflect}" grasp="${finger_grasp}">
        <origin rpy="0 0 0" xyz="0.0 ${reflect*finger_width} ${finger_length}"/>

File: intera_tools_description/urdf/electric_gripper/rethink_electric_gripper.xacro (robot description, xacro)
@@ -8,5 +8,5 @@
         <origin rpy="${-pi/2} ${pi} 0" xyz="0 0 0"/>
         <geometry>
-          <mesh filename="package://rethink_ee_description/meshes/electric_gripper/electric_gripper_base.DAE"/>
+          <mesh filename="package://intera_tools_description/meshes/electric_gripper/electric_gripper_base.DAE"/>
         </geometry>
       </visual>
@@ -28,9 +28,9 @@
     <!-- Left finger link -->
     <xacro:property name="finger_length" value="0.0" scope="global"/>
-    <xacro:include filename="$(find rethink_ee_description)/urdf/electric_gripper/fingers/${l_finger}.xacro" />
+    <xacro:include filename="$(find intera_tools_description)/urdf/electric_gripper/fingers/${l_finger}.xacro" />
     <xacro:finger_xacro gripper_side="${gripper_side}" finger_side="l" reflect="1" finger_tip="${l_finger_tip}" finger_grasp="${l_finger_grasp}"/>
     <xacro:property name="tip_finger_length" value="${finger_length}" scope="local"/>
     <!-- Right finger link -->
-    <xacro:include filename="$(find rethink_ee_description)/urdf/electric_gripper/fingers/${r_finger}.xacro" />
+    <xacro:include filename="$(find intera_tools_description)/urdf/electric_gripper/fingers/${r_finger}.xacro" />
     <xacro:finger_xacro gripper_side="${gripper_side}" finger_side="r" reflect="-1" finger_tip="${r_finger_tip}" finger_grasp="${r_finger_grasp}"/>
     <xacro:if value="${finger_length > tip_finger_length}">

File: intera_tools_description/urdf/null_gripper/example_end_effector.urdf.xacro (robot description, xacro)
@@ -1,5 +1,5 @@
 <?xml version="1.0"?>
 <robot xmlns:xacro="http://www.ros.org/wiki/xacro" name="left_null_gripper">
-  <xacro:include filename="$(find rethink_ee_description)/urdf/null_gripper/null_gripper.xacro" />
+  <xacro:include filename="$(find intera_tools_description)/urdf/null_gripper/null_gripper.xacro" />
   <xacro:null_gripper side="left"/>
 </robot>

File: intera_tools_description/urdf/pneumatic_gripper/example_end_effector.urdf.xacro (robot description, xacro)
@@ -1,5 +1,5 @@
 <?xml version="1.0"?>
 <robot xmlns:xacro="http://www.ros.org/wiki/xacro" name="left_pneumatic_gripper">
-  <xacro:include filename="$(find rethink_ee_description)/urdf/electric_gripper/rethink_pneumatic_gripper.xacro" />
+  <xacro:include filename="$(find intera_tools_description)/urdf/electric_gripper/rethink_pneumatic_gripper.xacro" />
   <xacro:rethink_pneumatic_gripper side="left"/>
 </robot>

File: intera_tools_description/urdf/pneumatic_gripper/pneumatic_gripper_base.xacro (robot description, xacro)
@@ -8,5 +8,5 @@
         <origin rpy="0 ${pi} ${pi}" xyz="0 0 0"/>
         <geometry>
-          <mesh filename="package://rethink_ee_description/meshes/pneumatic_gripper/pneumatic_gripper_base.DAE"/>
+          <mesh filename="package://intera_tools_description/meshes/pneumatic_gripper/pneumatic_gripper_base.DAE"/>
         </geometry>
       </visual>

File: intera_tools_description/urdf/pneumatic_gripper/rethink_pneumatic_gripper.xacro (robot description, xacro)
@@ -8,5 +8,5 @@
         <origin rpy="0 ${pi} ${pi}" xyz="0 0 0"/>
         <geometry>
-          <mesh filename="package://rethink_ee_description/meshes/pneumatic_gripper/pneumatic_gripper_w_cup.DAE"/>
+          <mesh filename="package://intera_tools_description/meshes/pneumatic_gripper/pneumatic_gripper_w_cup.DAE"/>
         </geometry>
       </visual>

Commit message: Sawyer Electric Gripper Update
- Adds connector_plate mesh and Xacro URDF
- Modifies electric gripper to accommodate connector plate
- Rotates electric gripper mesh and collision shape
- Uses new {side}_electric_gripper_base link as meshes link
- Uses {side}_gripper_base for complete end effector base link
- Updated offset for to center electric gripper finger joints
- URDF Config msg update for XML fragments
- Adds .gitignore for linux & blender files
- Adds smart_tool_plate mesh

File: intera_tools_description/urdf/electric_gripper/example_end_effector.urdf.xacro (robot description, xacro)
@@ -1,13 +1,14 @@
 <?xml version="1.0"?>
-<robot xmlns:xacro="http://www.ros.org/wiki/xacro" name="left_electric_gripper">
+<robot xmlns:xacro="http://www.ros.org/wiki/xacro" name="right_electric_gripper">
   <xacro:include filename="$(find intera_tools_description)/urdf/electric_gripper/rethink_electric_gripper.xacro" />
-  <xacro:rethink_electric_gripper side="left"
-                                  l_finger="extended_narrow"
+  <xacro:rethink_electric_gripper side="right"
+                                  l_finger="standard_narrow"
                                   l_finger_slot="2"
-                                  l_finger_tip="paddle_tip"
+                                  l_finger_tip="basic_hard_tip"
                                   l_finger_grasp="inner"
-                                  r_finger="extended_narrow"
+                                  r_finger="standard_narrow"
                                   r_finger_slot="2"
                                   r_finger_tip="basic_hard_tip"
-                                  r_finger_grasp="inner"/>
+                                  r_finger_grasp="inner"
+                                  use_connector_plate="True"/>
 </robot>

File: intera_tools_description/urdf/electric_gripper/rethink_electric_gripper.xacro (robot description, xacro)
@@ -1,10 +1,18 @@
 <?xml version="1.0"?>
 <robot xmlns:xacro="http://www.ros.org/wiki/xacro" name="rethink_electric_gripper">
-  <xacro:macro name="rethink_electric_gripper" params="side r_finger r_finger_slot r_finger_tip r_finger_grasp l_finger l_finger_slot l_finger_tip l_finger_grasp">
+  <xacro:macro name="rethink_electric_gripper" params="side r_finger r_finger_slot r_finger_tip r_finger_grasp l_finger l_finger_slot l_finger_tip l_finger_grasp use_connector_plate">
     <xacro:property name="gripper_side" value="${side[0]}" scope="local"/>
     <!-- Base of end effector -->
     <link name="${side}_gripper_base">
+      <inertial>
+        <origin rpy="0 0 0" xyz="0 0 0"/>
+        <mass value="0.0001"/>
+        <inertia ixx="0" ixy="0" ixz="0" iyy="0" iyz="0" izz="0.0"/>
+      </inertial>
+    </link>
+    <!-- Electric Gripper Base Link -->
+    <link name="${side}_electric_gripper_base">
       <visual>
-        <origin rpy="${-pi/2} ${pi} 0" xyz="0 0 0"/>
+        <origin rpy="0 0 0" xyz="0 0 0"/>
         <geometry>
           <mesh filename="package://intera_tools_description/meshes/electric_gripper/electric_gripper_base.DAE"/>
@@ -12,5 +20,5 @@
       </visual>
       <collision>
-        <origin rpy="${-pi/2} ${pi} 0" xyz="0.0 0.0 0"/>
+        <origin rpy="${-pi/2} ${pi} 0" xyz="0.004 0.0 0.025"/>
         <geometry>
           <cylinder length="0.1" radius="0.029"/>
@@ -22,8 +30,32 @@
       <inertial>
         <origin rpy="${-pi/2} ${pi} 0" xyz="0.0 0.0 0.0"/>
+        <!-- gripper_base mass -->
         <mass value="0.3"/>
         <inertia ixx="2e-08" ixy="0" ixz="0" iyy="3e-08" iyz="0" izz="2e-08"/>
       </inertial>
     </link>
+   <xacro:unless value="${use_connector_plate}">
+     <xacro:property name="electric_gripper_parent_link" value="${side}_gripper_base" scope="local"/>
+     <xacro:property name="connector_plate_length" value="0.0" scope="local"/>
+   </xacro:unless>
+   <xacro:if value="${use_connector_plate}">
+     <!-- Connector Plate Joint -->
+     <joint name="${side}_connector_plate_joint" type="fixed">
+       <origin xyz="0 0 0" rpy="0 0 0" />
+       <parent link="${side}_gripper_base"  />
+       <child  link="${side}_connector_plate_base" />
+     </joint>
+     <!-- Connector Plate Link -->
+     <xacro:include filename="$(find intera_tools_description)/urdf/connector_plate/connector_plate.xacro" />
+     <xacro:rethink_connector_plate side="${side}"/>
+     <xacro:property name="electric_gripper_parent_link" value="${side}_connector_plate_mount" scope="local"/>
+     <xacro:property name="connector_plate_length" value="${rethink_connector_plate_length}" scope="local"/>
+   </xacro:if>
+   <!-- Electric Gripper Base joint -->
+    <joint name="${side}_electric_gripper_base_jnt" type="fixed">
+      <origin rpy="0 0 0" xyz="0 0 0"/>
+      <parent link="${electric_gripper_parent_link}"/>
+      <child link="${side}_electric_gripper_base"/>
+    </joint>
     <!-- Left finger link -->
     <xacro:property name="finger_length" value="0.0" scope="global"/>
@@ -37,13 +69,14 @@
         <xacro:property name="tip_finger_length" value="${finger_length}" scope="local"/>
     </xacro:if>
-    <!-- Electric Gripper Base Joint -->
+    <!-- Gripper Base Joint -->
     <joint name="${side}_gripper_base" type="fixed">
-      <origin rpy="0 0 0" xyz="0 0 0.025"/>
+      <origin rpy="0 0 0" xyz="0 0 0"/>
       <parent link="${side}_hand"/>
       <child link="${side}_gripper_base"/>
     </joint>
-    <!-- Electric Gripper Tip joint -->
+    <!-- Gripper Tip joint -->
+   <xacro:property name="electric_gripper_base_length" value="0.04552" scope="local"/>
     <joint name="${side}_endpoint" type="fixed">
-      <origin rpy="0 0 0" xyz="0 0 ${tip_finger_length+0.02}"/>
+      <origin rpy="0 0 0" xyz="0 0 ${connector_plate_length+electric_gripper_base_length+tip_finger_length}"/>
       <parent link="${side}_gripper_base"/>
       <child link="${side}_gripper"/>
@@ -60,7 +93,7 @@
     <xacro:property name="l_finger_offset" value="${((l_finger_slot-1)*0.0095) -0.011}" scope="local"/>
     <joint name="${gripper_side}_gripper_l_finger_joint" type="prismatic">
-      <origin rpy="0 0 0" xyz="0.0 ${l_finger_offset} 0.02"/>
+      <origin rpy="0 0 0" xyz="0.003 ${l_finger_offset} ${electric_gripper_base_length}"/>
       <axis xyz="0 1 0"/>
-      <parent link="${side}_gripper_base"/>
+      <parent link="${side}_electric_gripper_base"/>
       <child link="${gripper_side}_gripper_l_finger"/>
       <limit effort="20.0" lower="0.0" upper="0.020833" velocity="5.0"/>
@@ -70,7 +103,7 @@
     <xacro:property name="r_finger_offset" value="${((r_finger_slot-1)*-0.0095) +0.011}" scope="local"/>
     <joint name="${gripper_side}_gripper_r_finger_joint" type="prismatic">
-      <origin rpy="0 0 0" xyz="0.0 ${r_finger_offset} 0.02"/>
+      <origin rpy="0 0 0" xyz="0.003 ${r_finger_offset} ${electric_gripper_base_length}"/>
       <axis xyz="0 1 0"/>
-      <parent link="${side}_gripper_base"/>
+      <parent link="${side}_electric_gripper_base"/>
       <child link="${gripper_side}_gripper_r_finger"/>
       <limit effort="20.0" lower="-0.020833" upper="0.0" velocity="5.0"/>
