Commit message: Update EPG Equivalent Inertia Sum for fingers

File: intera_tools_description/urdf/electric_gripper/rethink_electric_gripper.xacro (robot description, xacro)
@@ -7,6 +7,6 @@
       <inertial>
         <!-- Sum Gripper Mass - for whole end effector, measured from end of plastic cuff -->
-        <mass value="0.44"/>
-        <origin rpy="0 0 0" xyz="0.0028 -0.0004 0.0322"/>
+        <mass value="0.47"/>
+        <origin rpy="0 0 0" xyz="0.0028 -0.0004 0.0343"/>
         <inertia ixx="1e-08" ixy="0" ixz="0" iyy="1e-08" iyz="0" izz="1e-08"/>
       </inertial>

Commit message: Added friction and damping for gripper joints

File: intera_tools_description/urdf/electric_gripper/rethink_electric_gripper.xacro (robot description, xacro)
@@ -99,5 +99,5 @@
       <child link="${gripper_side}_gripper_l_finger"/>
       <limit effort="20.0" lower="0.0" upper="0.020833" velocity="5.0"/>
-      <dynamics damping="0.7" friction="0.0"/>
+      <dynamics damping="1000.0" friction="5000.0"/>
     </joint>
     <!-- Right finger -->
@@ -110,5 +110,5 @@
       <limit effort="20.0" lower="-0.020833" upper="0.0" velocity="5.0"/>
       <mimic joint="${gripper_side}_gripper_l_finger_joint" multiplier="-1.0"/>
-      <dynamics damping="0.7" friction="0.0"/>
+      <dynamics damping="1000.0" friction="5000.0"/>
     </joint>
     <xacro:if value="${gazebo}">
