Commit message: fixed bug in none fingertip

File: intera_tools_description/urdf/electric_gripper/fingers/none.xacro (robot description, xacro)
@@ -1,5 +1,5 @@
 <?xml version="1.0"?>
 <robot xmlns:xacro="http://www.ros.org/wiki/xacro" name="none_tip">
-  <xacro:macro name="finger_tip_xacro" params="parent_link reflect *joint_origin">
+  <xacro:macro name="finger_tip_xacro" params="parent_link grip reflect *joint_origin">
     <link name="${parent_link}_tip">
     </link>
