Commit message: Update Zero mass for gazebo, remove tip collision
* Modify inertial "zero" values to be very small values:
  - 1.1e-9 for inertia and 2e-6 for mass
* Remove tip collision (visual is still in robot's default epg config)

File: intera_tools_description/urdf/electric_gripper/fingers/basic_hard_tip.xacro (robot description, xacro)
@@ -20,7 +20,7 @@
       </collision>
       <inertial>
-        <origin rpy="0 0 0" xyz="0 0 0"/>
-        <mass value="0.0"/>
-        <inertia ixx="0.01" ixy="0" ixz="0" iyy="0.01" iyz="0" izz="0.01"/>
+        <origin rpy="0 0 ${pi*(g_reflect+1)/2}" xyz="0 0 0"/>
+        <mass value="2e-06"/>
+        <inertia ixx="1.1e-09" ixy="0" ixz="0" iyy="1.1e-09" iyz="0" izz="1.1e-09"/>
       </inertial>
     </link>

File: intera_tools_description/urdf/electric_gripper/fingers/basic_soft_tip.xacro (robot description, xacro)
@@ -20,7 +20,7 @@
       </collision>
       <inertial>
-        <origin rpy="0 0 0" xyz="0 0 0"/>
-        <mass value="0.0"/>
-        <inertia ixx="0.01" ixy="0" ixz="0" iyy="0.01" iyz="0" izz="0.01"/>
+        <origin rpy="0 0 ${pi*(g_reflect+1)/2}" xyz="0 0 0"/>
+        <mass value="2e-06"/>
+        <inertia ixx="1.1e-09" ixy="0" ixz="0" iyy="1.1e-09" iyz="0" izz="1.1e-09"/>
       </inertial>
     </link>

File: intera_tools_description/urdf/electric_gripper/fingers/extended_narrow.xacro (robot description, xacro)
@@ -30,7 +30,7 @@
       </collision>
       <inertial>
-        <origin rpy="0 0 0" xyz="0 0 0"/>
-        <mass value="0.0"/>
-        <inertia ixx="0.01" ixy="0" ixz="0" iyy="0.01" iyz="0" izz="0.01"/>
+        <origin rpy="0 0 ${-pi/2*(reflect+1)}" xyz="0 0 0"/>
+        <mass value="2e-06"/>
+        <inertia ixx="1.1e-09" ixy="0" ixz="0" iyy="1.1e-09" iyz="0" izz="1.1e-09"/>
       </inertial>
     </link>

File: intera_tools_description/urdf/electric_gripper/fingers/extended_wide.xacro (robot description, xacro)
@@ -30,7 +30,7 @@
       </collision>
       <inertial>
-        <origin rpy="0 0 0" xyz="0 0 0"/>
-        <mass value="0.0"/>
-        <inertia ixx="0.01" ixy="0" ixz="0" iyy="0.01" iyz="0" izz="0.01"/>
+        <origin rpy="0 0 ${-pi/2*(reflect+1)}" xyz="0 0 0"/>
+        <mass value="2e-06"/>
+        <inertia ixx="1.1e-09" ixy="0" ixz="0" iyy="1.1e-09" iyz="0" izz="1.1e-09"/>
       </inertial>
     </link>

File: intera_tools_description/urdf/electric_gripper/fingers/half_round_tip.xacro (robot description, xacro)
@@ -20,7 +20,7 @@
       </collision>
       <inertial>
-        <origin rpy="0 0 0" xyz="0 0 0"/>
-        <mass value="0.0"/>
-        <inertia ixx="0.01" ixy="0" ixz="0" iyy="0.01" iyz="0" izz="0.01"/>
+        <origin rpy="0 0 ${pi*(g_reflect+1)/2}" xyz="0 0 0"/>
+        <mass value="2e-06"/>
+        <inertia ixx="1.1e-09" ixy="0" ixz="0" iyy="1.1e-09" iyz="0" izz="1.1e-09"/>
       </inertial>
     </link>

File: intera_tools_description/urdf/electric_gripper/fingers/paddle_tip.xacro (robot description, xacro)
@@ -20,7 +20,7 @@
       </collision>
       <inertial>
-        <origin rpy="0 0 0" xyz="0 0 0"/>
-        <mass value="0.0"/>
-        <inertia ixx="0.01" ixy="0" ixz="0" iyy="0.01" iyz="0" izz="0.01"/>
+        <origin rpy="0 0 ${pi*(g_reflect+1)/2}" xyz="0 0 0"/>
+        <mass value="2e-06"/>
+        <inertia ixx="1.1e-09" ixy="0" ixz="0" iyy="1.1e-09" iyz="0" izz="1.1e-09"/>
       </inertial>
     </link>

File: intera_tools_description/urdf/electric_gripper/fingers/standard_narrow.xacro (robot description, xacro)
@@ -30,7 +30,7 @@
       </collision>
       <inertial>
-        <origin rpy="0 0 0" xyz="0 0 0"/>
-        <mass value="0.0"/>
-        <inertia ixx="0.01" ixy="0" ixz="0" iyy="0.01" iyz="0" izz="0.01"/>
+        <origin rpy="0 0 ${-pi/2*(reflect+1)}" xyz="0 0 0"/>
+        <mass value="2e-06"/>
+        <inertia ixx="1.1e-09" ixy="0" ixz="0" iyy="1.1e-09" iyz="0" izz="1.1e-09"/>
       </inertial>
     </link>

File: intera_tools_description/urdf/electric_gripper/fingers/standard_wide.xacro (robot description, xacro)
@@ -30,7 +30,7 @@
       </collision>
       <inertial>
-        <origin rpy="0 0 0" xyz="0 0 0"/>
-        <mass value="0.0"/>
-        <inertia ixx="0.01" ixy="0" ixz="0" iyy="0.01" iyz="0" izz="0.01"/>
+        <origin rpy="0 0 ${-pi/2*(reflect+1)}" xyz="0 0 0"/>
+        <mass value="2e-06"/>
+        <inertia ixx="1.1e-09" ixy="0" ixz="0" iyy="1.1e-09" iyz="0" izz="1.1e-09"/>
       </inertial>
     </link>

File: intera_tools_description/urdf/electric_gripper/rethink_electric_gripper.xacro (robot description, xacro)
@@ -31,6 +31,6 @@
       <inertial>
         <origin rpy="${-pi/2} ${pi} 0" xyz="0.0 0.0 0.0"/>
-        <mass value="0.0"/>
-        <inertia ixx="1e-08" ixy="0" ixz="0" iyy="1e-08" iyz="0" izz="1e-08"/>
+        <mass value="2e-06"/>
+        <inertia ixx="1.1e-09" ixy="0" ixz="0" iyy="1.1e-09" iyz="0" izz="1.1e-09"/>
       </inertial>
     </link>
@@ -86,23 +86,8 @@
     <link name="${side}_gripper_tip">
       <inertial>
-        <origin rpy="0 0 0" xyz="0 0 0"/>
-        <mass value="0.0001"/>
-        <inertia ixx="0" ixy="0" ixz="0" iyy="0" iyz="0" izz="0.0"/>
+        <origin xyz="0 0 0" rpy="0 0 0"/>
+        <mass value="2e-06"/>
+        <inertia ixx="1.1e-09" ixy="0" ixz="0" iyy="1.1e-09" iyz="0" izz="1.1e-09"/>
       </inertial>
-      <visual>
-        <origin xyz="0 0 0" rpy="0 0 0" />
-        <geometry>
-          <box size="0.015 0.015 0.015"/>
-        </geometry>
-        <material name="darkgrey">
-          <color rgba="0.2 0.3 0.3 1" />
-        </material>
-      </visual>
-      <collision>
-        <origin xyz="0 0 0" rpy="0 0 0" />
-        <geometry>
-          <box size="0.01 0.01 0.01"/>
-        </geometry>
-      </collision>
     </link>
     <!-- Left finger -->

Commit message: Minimal viable masses and inertias for Gazebo

File: intera_tools_description/urdf/electric_gripper/fingers/basic_hard_tip.xacro (robot description, xacro)
@@ -21,6 +21,6 @@
       <inertial>
         <origin rpy="0 0 ${pi*(g_reflect+1)/2}" xyz="0 0 0"/>
-        <mass value="2e-06"/>
-        <inertia ixx="1.1e-09" ixy="0" ixz="0" iyy="1.1e-09" iyz="0" izz="1.1e-09"/>
+        <mass value="0.001"/>
+        <inertia ixx="0.01" ixy="0" ixz="0" iyy="0.01" iyz="0" izz="0.01"/>
       </inertial>
     </link>

File: intera_tools_description/urdf/electric_gripper/fingers/basic_soft_tip.xacro (robot description, xacro)
@@ -21,6 +21,6 @@
       <inertial>
         <origin rpy="0 0 ${pi*(g_reflect+1)/2}" xyz="0 0 0"/>
-        <mass value="2e-06"/>
-        <inertia ixx="1.1e-09" ixy="0" ixz="0" iyy="1.1e-09" iyz="0" izz="1.1e-09"/>
+        <mass value="0.001"/>
+        <inertia ixx="0.01" ixy="0" ixz="0" iyy="0.01" iyz="0" izz="0.01"/>
       </inertial>
     </link>

File: intera_tools_description/urdf/electric_gripper/fingers/extended_narrow.xacro (robot description, xacro)
@@ -31,6 +31,6 @@
       <inertial>
         <origin rpy="0 0 ${-pi/2*(reflect+1)}" xyz="0 0 0"/>
-        <mass value="2e-06"/>
-        <inertia ixx="1.1e-09" ixy="0" ixz="0" iyy="1.1e-09" iyz="0" izz="1.1e-09"/>
+        <mass value="0.001"/>
+        <inertia ixx="0.01" ixy="0" ixz="0" iyy="0.01" iyz="0" izz="0.01"/>
       </inertial>
     </link>

File: intera_tools_description/urdf/electric_gripper/fingers/extended_wide.xacro (robot description, xacro)
@@ -31,6 +31,6 @@
       <inertial>
         <origin rpy="0 0 ${-pi/2*(reflect+1)}" xyz="0 0 0"/>
-        <mass value="2e-06"/>
-        <inertia ixx="1.1e-09" ixy="0" ixz="0" iyy="1.1e-09" iyz="0" izz="1.1e-09"/>
+        <mass value="0.001"/>
+        <inertia ixx="0.01" ixy="0" ixz="0" iyy="0.01" iyz="0" izz="0.01"/>
       </inertial>
     </link>

File: intera_tools_description/urdf/electric_gripper/fingers/half_round_tip.xacro (robot description, xacro)
@@ -21,6 +21,6 @@
       <inertial>
         <origin rpy="0 0 ${pi*(g_reflect+1)/2}" xyz="0 0 0"/>
-        <mass value="2e-06"/>
-        <inertia ixx="1.1e-09" ixy="0" ixz="0" iyy="1.1e-09" iyz="0" izz="1.1e-09"/>
+        <mass value="0.001"/>
+        <inertia ixx="0.01" ixy="0" ixz="0" iyy="0.01" iyz="0" izz="0.01"/>
       </inertial>
     </link>

File: intera_tools_description/urdf/electric_gripper/fingers/paddle_tip.xacro (robot description, xacro)
@@ -21,6 +21,6 @@
       <inertial>
         <origin rpy="0 0 ${pi*(g_reflect+1)/2}" xyz="0 0 0"/>
-        <mass value="2e-06"/>
-        <inertia ixx="1.1e-09" ixy="0" ixz="0" iyy="1.1e-09" iyz="0" izz="1.1e-09"/>
+        <mass value="0.001"/>
+        <inertia ixx="0.01" ixy="0" ixz="0" iyy="0.01" iyz="0" izz="0.01"/>
       </inertial>
     </link>

File: intera_tools_description/urdf/electric_gripper/fingers/standard_narrow.xacro (robot description, xacro)
@@ -31,6 +31,6 @@
       <inertial>
         <origin rpy="0 0 ${-pi/2*(reflect+1)}" xyz="0 0 0"/>
-        <mass value="2e-06"/>
-        <inertia ixx="1.1e-09" ixy="0" ixz="0" iyy="1.1e-09" iyz="0" izz="1.1e-09"/>
+        <mass value="0.001"/>
+        <inertia ixx="0.01" ixy="0" ixz="0" iyy="0.01" iyz="0" izz="0.01"/>
       </inertial>
     </link>

File: intera_tools_description/urdf/electric_gripper/fingers/standard_wide.xacro (robot description, xacro)
@@ -31,6 +31,6 @@
       <inertial>
         <origin rpy="0 0 ${-pi/2*(reflect+1)}" xyz="0 0 0"/>
-        <mass value="2e-06"/>
-        <inertia ixx="1.1e-09" ixy="0" ixz="0" iyy="1.1e-09" iyz="0" izz="1.1e-09"/>
+        <mass value="0.001"/>
+        <inertia ixx="0.01" ixy="0" ixz="0" iyy="0.01" iyz="0" izz="0.01"/>
       </inertial>
     </link>

File: intera_tools_description/urdf/electric_gripper/rethink_electric_gripper.xacro (robot description, xacro)
@@ -99,5 +99,5 @@
       <child link="${gripper_side}_gripper_l_finger"/>
       <limit effort="20.0" lower="0.0" upper="0.020833" velocity="5.0"/>
-      <dynamics damping="1000.0" friction="5000.0"/>
+      <dynamics damping="100.0" friction="500.0"/>
     </joint>
     <!-- Right finger -->
@@ -110,5 +110,5 @@
       <limit effort="20.0" lower="-0.020833" upper="0.0" velocity="5.0"/>
       <mimic joint="${gripper_side}_gripper_l_finger_joint" multiplier="-1.0"/>
-      <dynamics damping="1000.0" friction="5000.0"/>
+      <dynamics damping="100.0" friction="500.0"/>
     </joint>
     <xacro:if value="${gazebo}">
