Commit message: Tweaks for the electric gripper

File: intera_tools_description/urdf/connector_plate/connector_plate.xacro (robot description, xacro)
@@ -31,5 +31,5 @@
   <link name="${side}_connector_plate_mount" />
   <joint name="${side}_connector_plate_base_joint" type="fixed">
-    <origin xyz="0 0 ${rethink_connector_plate_length}" rpy="0 0 0" />
+    <origin xyz="0 0 ${rethink_connector_plate_length+0.0025}" rpy="0 0 0" />
     <parent link="${side}_connector_plate_base"  />
     <child  link="${side}_connector_plate_mount" />

File: intera_tools_description/urdf/electric_gripper/rethink_electric_gripper.xacro (robot description, xacro)
@@ -42,5 +42,5 @@
      <!-- Connector Plate Joint -->
      <joint name="${side}_connector_plate_joint" type="fixed">
-       <origin xyz="0 0 0" rpy="0 0 0" />
+       <origin xyz="0 0 -0.0032" rpy="0 0 0" />
        <parent link="${side}_gripper_base"  />
        <child  link="${side}_connector_plate_base" />

Commit message: Updates for connector_plate mesh color

File: intera_tools_description/urdf/connector_plate/connector_plate.xacro (robot description, xacro)
@@ -1,5 +1,5 @@
 <?xml version="1.0"?>
 <robot xmlns:xacro="http://www.ros.org/wiki/xacro" name="rethink_connector_plate">
-  <xacro:macro name="rethink_connector_plate" params="side">
+  <xacro:macro name="rethink_connector_plate" params="side gazebo">
   <xacro:property name="rethink_connector_plate_length" value="0.0151" scope="global"/>
   <link name="${side}_connector_plate_base">
@@ -29,4 +29,9 @@
     </collision>
   </link>
+  <xacro:if value="${gazebo}">
+    <gazebo reference="${side}_connector_plate_base">
+      <material>Gazebo/FlatBlack</material>
+    </gazebo>
+  </xacro:if>
   <link name="${side}_connector_plate_mount" />
   <joint name="${side}_connector_plate_base_joint" type="fixed">

File: intera_tools_description/urdf/electric_gripper/rethink_electric_gripper.xacro (robot description, xacro)
@@ -1,5 +1,5 @@
 <?xml version="1.0"?>
 <robot xmlns:xacro="http://www.ros.org/wiki/xacro" name="rethink_electric_gripper">
-  <xacro:macro name="rethink_electric_gripper" params="side r_finger r_finger_slot r_finger_tip r_finger_grasp l_finger l_finger_slot l_finger_tip l_finger_grasp use_connector_plate">
+  <xacro:macro name="rethink_electric_gripper" params="side r_finger r_finger_slot r_finger_tip r_finger_grasp l_finger l_finger_slot l_finger_tip l_finger_grasp use_connector_plate gazebo">
     <xacro:property name="gripper_side" value="${side[0]}" scope="local"/>
     <!-- Base of end effector -->
@@ -48,5 +48,5 @@
      <!-- Connector Plate Link -->
      <xacro:include filename="$(find intera_tools_description)/urdf/connector_plate/connector_plate.xacro" />
-     <xacro:rethink_connector_plate side="${side}"/>
+     <xacro:rethink_connector_plate side="${side}" gazebo="${gazebo}"/>
      <xacro:property name="electric_gripper_parent_link" value="${side}_connector_plate_mount" scope="local"/>
      <xacro:property name="connector_plate_length" value="${rethink_connector_plate_length}" scope="local"/>
@@ -111,11 +111,12 @@
       <dynamics damping="0.7" friction="0.0"/>
     </joint>
+    <xacro:if value="${gazebo}">
     <transmission name="gripper_${side}1">
       <type>transmission_interface/SimpleTransmission</type>
       <joint name="${gripper_side}_gripper_r_finger_joint">
-        <hardwareInterface>EffortJointInterface</hardwareInterface>
+        <hardwareInterface>hardware_interface/EffortJointInterface</hardwareInterface>
       </joint>
       <actuator name="gripper_${gripper_side}1_motor1">
-        <hardwareInterface>EffortJointInterface</hardwareInterface>
+        <hardwareInterface>hardware_interface/EffortJointInterface</hardwareInterface>
         <mechanicalReduction>1</mechanicalReduction>
       </actuator>
@@ -124,8 +125,8 @@
       <type>transmission_interface/SimpleTransmission</type>
       <joint name="${gripper_side}_gripper_l_finger_joint">
-        <hardwareInterface>EffortJointInterface</hardwareInterface>
+        <hardwareInterface>hardware_interface/EffortJointInterface</hardwareInterface>
       </joint>
       <actuator name="gripper_${gripper_side}1_motor2">
-        <hardwareInterface>EffortJointInterface</hardwareInterface>
+        <hardwareInterface>hardware_interface/EffortJointInterface</hardwareInterface>
         <mechanicalReduction>1</mechanicalReduction>
       </actuator>
@@ -137,4 +138,5 @@
       <implicitSpringDamper>1</implicitSpringDamper>
     </gazebo>
+    </xacro:if>
   </xacro:macro>
 </robot>

Commit message: Update EPG xacro and remove per-link inertias
Synchronizes the structure and naming of the EPG xacro w/ upstream.

Also remove the per-links masses and inertias (for now).

File: intera_tools_description/urdf/connector_plate/connector_plate.xacro (robot description, xacro)
@@ -5,6 +5,6 @@
   <link name="${side}_connector_plate_base">
     <inertial>
-      <origin xyz="-0.00032768 -2.5612E-05 0.0062193" rpy="0 0 0" />
-      <mass value="0.1609" />
+      <origin xyz="0 0 0" rpy="0 0 0" />
+      <mass value="0.0" />
       <inertia ixx="6.9922E-05"  ixy="6.1026E-08"  ixz="-1.7042E-06"
                iyy="6.8188E-05"  iyz="-1.6118E-08" izz="0.00012392" />
@@ -35,5 +35,5 @@
   </xacro:if>
   <link name="${side}_connector_plate_mount" />
-  <joint name="${side}_connector_plate_base_joint" type="fixed">
+  <joint name="${side}_connector_plate_mount_joint" type="fixed">
     <origin xyz="0 0 ${rethink_connector_plate_length+0.0025}" rpy="0 0 0" />
     <parent link="${side}_connector_plate_base"  />

File: intera_tools_description/urdf/electric_gripper/fingers/basic_hard_tip.xacro (robot description, xacro)
@@ -20,6 +20,6 @@
       </collision>
       <inertial>
-        <origin rpy="0 0 ${pi*(g_reflect+1)/2}" xyz="0 0 0"/>
-        <mass value="0.01"/>
+        <origin rpy="0 0 0" xyz="0 0 0"/>
+        <mass value="0.0"/>
         <inertia ixx="0.01" ixy="0" ixz="0" iyy="0.01" iyz="0" izz="0.01"/>
       </inertial>

File: intera_tools_description/urdf/electric_gripper/fingers/basic_soft_tip.xacro (robot description, xacro)
@@ -20,6 +20,6 @@
       </collision>
       <inertial>
-        <origin rpy="0 0 ${pi*(g_reflect+1)/2}" xyz="0 0 0"/>
-        <mass value="0.01"/>
+        <origin rpy="0 0 0" xyz="0 0 0"/>
+        <mass value="0.0"/>
         <inertia ixx="0.01" ixy="0" ixz="0" iyy="0.01" iyz="0" izz="0.01"/>
       </inertial>

File: intera_tools_description/urdf/electric_gripper/fingers/extended_narrow.xacro (robot description, xacro)
@@ -1,5 +1,5 @@
 <?xml version="1.0"?>
 <robot xmlns:xacro="http://www.ros.org/wiki/xacro" name="extended_narrow">
-  <xacro:macro name="finger_xacro" params="gripper_side finger_side reflect finger_tip finger_grasp">
+  <xacro:macro name="finger_xacro" params="gripper_side finger_side reflect finger_tip finger_grasp gazebo">
   <xacro:property name="finger_length" value="0.1127" scope="global"/>
   <xacro:property name="finger_width" value="0.01725" scope="local"/>
@@ -30,24 +30,26 @@
       </collision>
       <inertial>
-        <origin rpy="0 0 ${-pi/2*(reflect+1)}" xyz="0 0 0"/>
-        <mass value="0.02"/>
+        <origin rpy="0 0 0" xyz="0 0 0"/>
+        <mass value="0.0"/>
         <inertia ixx="0.01" ixy="0" ixz="0" iyy="0.01" iyz="0" izz="0.01"/>
       </inertial>
     </link>
-    <gazebo reference="${gripper_side}_gripper_${finger_side}_finger">
-      <mu1>1000</mu1>
-      <mu2>1000</mu2>
-      <fdir1>0.0 0.0 1.0</fdir1>
-      <kp>1e5</kp>
-      <kd>1.0</kd>
-    </gazebo>
-   <xacro:property name="none" value="[none, false, null, empty]" scope="local"/>
-   <xacro:if value="${finger_tip in none}">
-     <xacro:property name="finger_tip" value="none" scope="local"/>
-   </xacro:if>
-   <xacro:include filename="$(find intera_tools_description)/urdf/electric_gripper/fingers/${finger_tip}.xacro" />
-   <xacro:finger_tip_xacro parent_link="${gripper_side}_gripper_${finger_side}_finger" reflect="${reflect}" grasp="${finger_grasp}">
-       <origin rpy="0 0 0" xyz="0.0 ${reflect*finger_width} ${finger_length}"/>
-   </xacro:finger_tip_xacro>
+    <xacro:if value="${gazebo}">
+      <gazebo reference="${gripper_side}_gripper_${finger_side}_finger">
+        <mu1>1000</mu1>
+        <mu2>1000</mu2>
+        <fdir1>0.0 0.0 1.0</fdir1>
+        <kp>1e5</kp>
+        <kd>1.0</kd>
+      </gazebo>
+    </xacro:if>
+    <xacro:property name="none" value="[none, false, null, empty]" scope="local"/>
+    <xacro:if value="${finger_tip in none}">
+      <xacro:property name="finger_tip" value="none" scope="local"/>
+    </xacro:if>
+    <xacro:include filename="$(find intera_tools_description)/urdf/electric_gripper/fingers/${finger_tip}.xacro" />
+    <xacro:finger_tip_xacro parent_link="${gripper_side}_gripper_${finger_side}_finger" reflect="${reflect}" grasp="${finger_grasp}">
+        <origin rpy="0 0 0" xyz="0.0 ${reflect*finger_width} ${finger_length}"/>
+    </xacro:finger_tip_xacro>
   </xacro:macro>
 </robot>

File: intera_tools_description/urdf/electric_gripper/fingers/extended_wide.xacro (robot description, xacro)
@@ -1,5 +1,5 @@
 <?xml version="1.0"?>
 <robot xmlns:xacro="http://www.ros.org/wiki/xacro" name="wide_extended">
-  <xacro:macro name="finger_xacro" params="gripper_side finger_side reflect finger_tip finger_grasp">
+  <xacro:macro name="finger_xacro" params="gripper_side finger_side reflect finger_tip finger_grasp gazebo">
     <xacro:property name="finger_length" value="0.1127" scope="global"/>
     <xacro:property name="finger_width" value="0.05503" scope="local"/>
@@ -30,24 +30,26 @@
       </collision>
       <inertial>
-        <origin rpy="0 0 ${-pi/2*(reflect+1)}" xyz="0 0 0"/>
-        <mass value="0.02"/>
+        <origin rpy="0 0 0" xyz="0 0 0"/>
+        <mass value="0.0"/>
         <inertia ixx="0.01" ixy="0" ixz="0" iyy="0.01" iyz="0" izz="0.01"/>
       </inertial>
     </link>
-    <gazebo reference="${gripper_side}_gripper_${finger_side}_finger">
-      <mu1>1000</mu1>
-      <mu2>1000</mu2>
-      <fdir1>0.0 0.0 1.0</fdir1>
-      <kp>1e5</kp>
-      <kd>1.0</kd>
-    </gazebo>
-   <xacro:property name="none" value="[none, false, null, empty]" scope="local"/>
-   <xacro:if value="${finger_tip in none}">
-     <xacro:property name="finger_tip" value="none" scope="local"/>
-   </xacro:if>
-   <xacro:include filename="$(find intera_tools_description)/urdf/electric_gripper/fingers/${finger_tip}.xacro" />
-   <xacro:finger_tip_xacro parent_link="${gripper_side}_gripper_${finger_side}_finger" reflect="${reflect}" grasp="${finger_grasp}">
-       <origin rpy="0 0 0" xyz="0.0 ${reflect*finger_width} ${finger_length}"/>
-   </xacro:finger_tip_xacro>
+    <xacro:if value="${gazebo}">
+      <gazebo reference="${gripper_side}_gripper_${finger_side}_finger">
+        <mu1>1000</mu1>
+        <mu2>1000</mu2>
+        <fdir1>0.0 0.0 1.0</fdir1>
+        <kp>1e5</kp>
+        <kd>1.0</kd>
+      </gazebo>
+    </xacro:if>
+    <xacro:property name="none" value="[none, false, null, empty]" scope="local"/>
+    <xacro:if value="${finger_tip in none}">
+      <xacro:property name="finger_tip" value="none" scope="local"/>
+    </xacro:if>
+    <xacro:include filename="$(find intera_tools_description)/urdf/electric_gripper/fingers/${finger_tip}.xacro" />
+    <xacro:finger_tip_xacro parent_link="${gripper_side}_gripper_${finger_side}_finger" reflect="${reflect}" grasp="${finger_grasp}">
+        <origin rpy="0 0 0" xyz="0.0 ${reflect*finger_width} ${finger_length}"/>
+    </xacro:finger_tip_xacro>
   </xacro:macro>
 </robot>

File: intera_tools_description/urdf/electric_gripper/fingers/half_round_tip.xacro (robot description, xacro)
@@ -20,6 +20,6 @@
       </collision>
       <inertial>
-        <origin rpy="0 0 ${pi*(g_reflect+1)/2}" xyz="0 0 0"/>
-        <mass value="0.01"/>
+        <origin rpy="0 0 0" xyz="0 0 0"/>
+        <mass value="0.0"/>
         <inertia ixx="0.01" ixy="0" ixz="0" iyy="0.01" iyz="0" izz="0.01"/>
       </inertial>

File: intera_tools_description/urdf/electric_gripper/fingers/paddle_tip.xacro (robot description, xacro)
@@ -20,6 +20,6 @@
       </collision>
       <inertial>
-        <origin rpy="0 0 ${pi*(g_reflect+1)/2}" xyz="0 0 0"/>
-        <mass value="0.01"/>
+        <origin rpy="0 0 0" xyz="0 0 0"/>
+        <mass value="0.0"/>
         <inertia ixx="0.01" ixy="0" ixz="0" iyy="0.01" iyz="0" izz="0.01"/>
       </inertial>

File: intera_tools_description/urdf/electric_gripper/fingers/standard_narrow.xacro (robot description, xacro)
@@ -1,5 +1,5 @@
 <?xml version="1.0"?>
 <robot xmlns:xacro="http://www.ros.org/wiki/xacro" name="standard_narrow">
-  <xacro:macro name="finger_xacro" params="gripper_side finger_side reflect finger_tip finger_grasp">
+  <xacro:macro name="finger_xacro" params="gripper_side finger_side reflect finger_tip finger_grasp gazebo">
   <xacro:property name="finger_length" value="0.075" scope="global"/>
   <xacro:property name="finger_width" value="0.01725" scope="local"/>
@@ -30,24 +30,26 @@
       </collision>
       <inertial>
-        <origin rpy="0 0 ${-pi/2*(reflect+1)}" xyz="0 0 0"/>
-        <mass value="0.02"/>
+        <origin rpy="0 0 0" xyz="0 0 0"/>
+        <mass value="0.0"/>
         <inertia ixx="0.01" ixy="0" ixz="0" iyy="0.01" iyz="0" izz="0.01"/>
       </inertial>
     </link>
-    <gazebo reference="${gripper_side}_gripper_${finger_side}_finger">
-      <mu1>1000</mu1>
-      <mu2>1000</mu2>
-      <fdir1>0.0 0.0 1.0</fdir1>
-      <kp>1e5</kp>
-      <kd>1.0</kd>
-    </gazebo>
-   <xacro:property name="none" value="[none, false, null, empty]" scope="local"/>
-   <xacro:if value="${finger_tip in none}">
-     <xacro:property name="finger_tip" value="none" scope="local"/>
-   </xacro:if>
-   <xacro:include filename="$(find intera_tools_description)/urdf/electric_gripper/fingers/${finger_tip}.xacro" />
-   <xacro:finger_tip_xacro parent_link="${gripper_side}_gripper_${finger_side}_finger" reflect="${reflect}" grasp="${finger_grasp}">
-       <origin rpy="0 0 0" xyz="0.0 ${reflect*finger_width} ${finger_length}"/>
-   </xacro:finger_tip_xacro>
+    <xacro:if value="${gazebo}">
+      <gazebo reference="${gripper_side}_gripper_${finger_side}_finger">
+        <mu1>1000</mu1>
+        <mu2>1000</mu2>
+        <fdir1>0.0 0.0 1.0</fdir1>
+        <kp>1e5</kp>
+        <kd>1.0</kd>
+      </gazebo>
+    </xacro:if>
+    <xacro:property name="none" value="[none, false, null, empty]" scope="local"/>
+    <xacro:if value="${finger_tip in none}">
+      <xacro:property name="finger_tip" value="none" scope="local"/>
+    </xacro:if>
+    <xacro:include filename="$(find intera_tools_description)/urdf/electric_gripper/fingers/${finger_tip}.xacro" />
+    <xacro:finger_tip_xacro parent_link="${gripper_side}_gripper_${finger_side}_finger" reflect="${reflect}" grasp="${finger_grasp}">
+        <origin rpy="0 0 0" xyz="0.0 ${reflect*finger_width} ${finger_length}"/>
+    </xacro:finger_tip_xacro>
   </xacro:macro>
 </robot>

File: intera_tools_description/urdf/electric_gripper/fingers/standard_wide.xacro (robot description, xacro)
@@ -1,5 +1,5 @@
 <?xml version="1.0"?>
 <robot xmlns:xacro="http://www.ros.org/wiki/xacro" name="standard_wide">
-  <xacro:macro name="finger_xacro" params="gripper_side finger_side reflect finger_tip finger_grasp">
+  <xacro:macro name="finger_xacro" params="gripper_side finger_side reflect finger_tip finger_grasp gazebo">
   <xacro:property name="finger_length" value="0.075" scope="global"/>
   <xacro:property name="finger_width" value="0.05503" scope="local"/>
@@ -30,24 +30,26 @@
       </collision>
       <inertial>
-        <origin rpy="0 0 ${-pi/2*(reflect+1)}" xyz="0 0 0"/>
-        <mass value="0.02"/>
+        <origin rpy="0 0 0" xyz="0 0 0"/>
+        <mass value="0.0"/>
         <inertia ixx="0.01" ixy="0" ixz="0" iyy="0.01" iyz="0" izz="0.01"/>
       </inertial>
     </link>
-    <gazebo reference="${gripper_side}_gripper_${finger_side}_finger">
-      <mu1>1000</mu1>
-      <mu2>1000</mu2>
-      <fdir1>0.0 0.0 1.0</fdir1>
-      <kp>1e5</kp>
-      <kd>1.0</kd>
-    </gazebo>
-   <xacro:property name="none" value="[none, false, null, empty]" scope="local"/>
-   <xacro:if value="${finger_tip in none}">
-     <xacro:property name="finger_tip" value="none" scope="local"/>
-   </xacro:if>
-   <xacro:include filename="$(find intera_tools_description)/urdf/electric_gripper/fingers/${finger_tip}.xacro" />
-   <xacro:finger_tip_xacro parent_link="${gripper_side}_gripper_${finger_side}_finger" reflect="${reflect}" grasp="${finger_grasp}">
-       <origin rpy="0 0 0" xyz="0.0 ${reflect*finger_width} ${finger_length}"/>
-   </xacro:finger_tip_xacro>
+    <xacro:if value="${gazebo}">
+      <gazebo reference="${gripper_side}_gripper_${finger_side}_finger">
+        <mu1>1000</mu1>
+        <mu2>1000</mu2>
+        <fdir1>0.0 0.0 1.0</fdir1>
+        <kp>1e5</kp>
+        <kd>1.0</kd>
+      </gazebo>
+    </xacro:if>
+    <xacro:property name="none" value="[none, false, null, empty]" scope="local"/>
+    <xacro:if value="${finger_tip in none}">
+      <xacro:property name="finger_tip" value="none" scope="local"/>
+    </xacro:if>
+    <xacro:include filename="$(find intera_tools_description)/urdf/electric_gripper/fingers/${finger_tip}.xacro" />
+    <xacro:finger_tip_xacro parent_link="${gripper_side}_gripper_${finger_side}_finger" reflect="${reflect}" grasp="${finger_grasp}">
+        <origin rpy="0 0 0" xyz="0.0 ${reflect*finger_width} ${finger_length}"/>
+    </xacro:finger_tip_xacro>
   </xacro:macro>
 </robot>

File: intera_tools_description/urdf/electric_gripper/rethink_electric_gripper.xacro (robot description, xacro)
@@ -2,11 +2,12 @@
 <robot xmlns:xacro="http://www.ros.org/wiki/xacro" name="rethink_electric_gripper">
   <xacro:macro name="rethink_electric_gripper" params="side r_finger r_finger_slot r_finger_tip r_finger_grasp l_finger l_finger_slot l_finger_tip l_finger_grasp use_connector_plate gazebo">
-    <xacro:property name="gripper_side" value="${side[0]}" scope="local"/>
-    <!-- Base of end effector -->
+    <xacro:property name="gripper_side" value="${side}" scope="local"/>
+    <!-- Base of whole end effector - (Connector Plate + Electric Gripper + Fingers + Tips) -->
     <link name="${side}_gripper_base">
       <inertial>
-        <origin rpy="0 0 0" xyz="0 0 0"/>
-        <mass value="0.0001"/>
-        <inertia ixx="0" ixy="0" ixz="0" iyy="0" iyz="0" izz="0.0"/>
+        <!-- Sum Gripper Mass - for whole end effector, measured from end of plastic cuff -->
+        <mass value="0.44"/>
+        <origin rpy="0 0 0" xyz="0.0028 -0.0004 0.0322"/>
+        <inertia ixx="1e-08" ixy="0" ixz="0" iyy="1e-08" iyz="0" izz="1e-08"/>
       </inertial>
     </link>
@@ -30,7 +31,6 @@
       <inertial>
         <origin rpy="${-pi/2} ${pi} 0" xyz="0.0 0.0 0.0"/>
-        <!-- gripper_base mass -->
-        <mass value="0.3"/>
-        <inertia ixx="2e-08" ixy="0" ixz="0" iyy="3e-08" iyz="0" izz="2e-08"/>
+        <mass value="0.0"/>
+        <inertia ixx="1e-08" ixy="0" ixz="0" iyy="1e-08" iyz="0" izz="1e-08"/>
       </inertial>
     </link>
@@ -41,6 +41,6 @@
    <xacro:if value="${use_connector_plate}">
      <!-- Connector Plate Joint -->
-     <joint name="${side}_connector_plate_joint" type="fixed">
-       <origin xyz="0 0 -0.0032" rpy="0 0 0" />
+     <joint name="${side}_connector_plate_base_joint" type="fixed">
+       <origin xyz="0 0 0.0018" rpy="0 0 0" />
        <parent link="${side}_gripper_base"  />
        <child  link="${side}_connector_plate_base" />
@@ -53,5 +53,5 @@
    </xacro:if>
    <!-- Electric Gripper Base joint -->
-    <joint name="${side}_electric_gripper_base_jnt" type="fixed">
+    <joint name="${side}_electric_gripper_base_joint" type="fixed">
       <origin rpy="0 0 0" xyz="0 0 0"/>
       <parent link="${electric_gripper_parent_link}"/>
@@ -61,27 +61,28 @@
     <xacro:property name="finger_length" value="0.0" scope="global"/>
     <xacro:include filename="$(find intera_tools_description)/urdf/electric_gripper/fingers/${l_finger}.xacro" />
-    <xacro:finger_xacro gripper_side="${gripper_side}" finger_side="l" reflect="1" finger_tip="${l_finger_tip}" finger_grasp="${l_finger_grasp}"/>
+    <xacro:finger_xacro gripper_side="${gripper_side}" finger_side="l" reflect="1" finger_tip="${l_finger_tip}" finger_grasp="${l_finger_grasp}" gazebo="${gazebo}"/>
     <xacro:property name="tip_finger_length" value="${finger_length}" scope="local"/>
     <!-- Right finger link -->
     <xacro:include filename="$(find intera_tools_description)/urdf/electric_gripper/fingers/${r_finger}.xacro" />
-    <xacro:finger_xacro gripper_side="${gripper_side}" finger_side="r" reflect="-1" finger_tip="${r_finger_tip}" finger_grasp="${r_finger_grasp}"/>
+    <xacro:finger_xacro gripper_side="${gripper_side}" finger_side="r" reflect="-1" finger_tip="${r_finger_tip}" finger_grasp="${r_finger_grasp}" gazebo="${gazebo}"/>
     <xacro:if value="${finger_length > tip_finger_length}">
         <xacro:property name="tip_finger_length" value="${finger_length}" scope="local"/>
     </xacro:if>
     <!-- Gripper Base Joint -->
-    <joint name="${side}_gripper_base" type="fixed">
-      <origin rpy="0 0 0" xyz="0 0 0"/>
+    <xacro:property name="end_of_arm_offset" value="-0.005" scope="local"/>
+    <joint name="${side}_gripper_base_joint" type="fixed">
+      <origin rpy="0 0 0" xyz="0 0 ${end_of_arm_offset}"/>
       <parent link="${side}_hand"/>
       <child link="${side}_gripper_base"/>
     </joint>
     <!-- Gripper Tip joint -->
-   <xacro:property name="electric_gripper_base_length" value="0.04552" scope="local"/>
-    <joint name="${side}_endpoint" type="fixed">
-      <origin rpy="0 0 0" xyz="0 0 ${connector_plate_length+electric_gripper_base_length+tip_finger_length}"/>
+    <xacro:property name="electric_gripper_base_length" value="0.04552" scope="local"/>
+    <joint name="${side}_gripper_tip_joint" type="fixed">
+      <origin rpy="0 0 0" xyz="0 0 ${(-1*end_of_arm_offset)+connector_plate_length+electric_gripper_base_length+tip_finger_length}"/>
       <parent link="${side}_gripper_base"/>
-      <child link="${side}_gripper"/>
+      <child link="${side}_gripper_tip"/>
     </joint>
     <!-- Electric Gripper Tip link -->
-    <link name="${side}_gripper">
+    <link name="${side}_gripper_tip">
       <inertial>
         <origin rpy="0 0 0" xyz="0 0 0"/>
@@ -89,4 +90,19 @@
         <inertia ixx="0" ixy="0" ixz="0" iyy="0" iyz="0" izz="0.0"/>
       </inertial>
+      <visual>
+        <origin xyz="0 0 0" rpy="0 0 0" />
+        <geometry>
+          <box size="0.015 0.015 0.015"/>
+        </geometry>
+        <material name="darkgrey">
+          <color rgba="0.2 0.3 0.3 1" />
+        </material>
+      </visual>
+      <collision>
+        <origin xyz="0 0 0" rpy="0 0 0" />
+        <geometry>
+          <box size="0.01 0.01 0.01"/>
+        </geometry>
+      </collision>
     </link>
     <!-- Left finger -->
