Commit message: Fix collision of connector_plate

File: intera_tools_description/urdf/connector_plate/connector_plate.xacro (robot description, xacro)
@@ -20,7 +20,7 @@
     </visual>
     <collision>
-      <origin xyz="0 0 0.0135" rpy="0 0 0" />
+      <origin xyz="0 0 ${rethink_connector_plate_length / 2}" rpy="0 0 0" />
         <geometry>
-          <cylinder length="${rethink_connector_plate_length*2.0}" radius="0.04"/>
+          <cylinder length="${rethink_connector_plate_length}" radius="0.04"/>
         </geometry>
         <material name="darkred">
